File: schematic/esp_controller.kicad_pcb (KiCad board)
At the start: 4 copper layers, 30.7 x 54.6 mm, 39 parts, among them J1 xt30, J2 jst_sh 6, J3 Conn_01x03, J4 Conn_01x03, J5 Conn_01x03, J6 Conn_01x03, J7 Screw_Terminal_01x06, Q1 FDN359BN, Q2 FDN359BN, Q3 FDN359BN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

Commit message: pcb second revision
Parts:
- added R6: 2k2, Resistor_SMD:R_0603_1608Metric, F.Cu at (240.0, 102.1)
- added R7: 2k2, Resistor_SMD:R_0603_1608Metric, F.Cu at (240.0, 100.5)
- added R8: 10k, Resistor_SMD:R_0603_1608Metric, F.Cu at (217.4, 96.5)
- added SW2: SW_SPST, Connector_PinHeader_1.27mm:PinHeader_1x02_P1.27mm_Vertical, F.Cu at (214.2, 97.3)
- R2: value 2.2k -> 2k2
- SW1: footprint Connector_PinHeader_2.54mm:PinHeader_1x02_P2.54mm_Vertical -> Connector_PinHeader_1.27mm:PinHeader_1x02_P1.27mm_Vertical
- moved C8 8.64 mm to (217.0, 113.1)
- moved SW1 3.29 mm to (241.8, 97.1)
- moved R2 1.90 mm to (216.1, 99.3), turned to 0 degrees
- moved R1 1.04 mm to (215.2, 101.9)
- moved R5 1.04 mm to (217.0, 101.9)
- moved R3 1.04 mm to (217.0, 106.4)
- moved J1 0.74 mm to (217.5, 123.1)
- moved C9 0.41 mm to (239.2, 110.8), turned to -90 degrees
- moved D1 0.30 mm to (221.8, 111.2), turned to 0 degrees
- moved D2 0.22 mm to (234.5, 111.2), turned to 0 degrees
- moved H1 0.21 mm to (214.9, 118.3)
- moved C5 0.19 mm to (240.6, 126.2)
- moved H3 0.10 mm to (241.0, 118.3)
Connections:
- D1 pad 2: Net-(D1-Pad2) -> unconnected-(D1-Pad2)
- D1 pad 4: /LED_TX -> Net-(D2-Pad2)
- D2 pad 2: unconnected-(D2-Pad2) -> Net-(D2-Pad2)
- D2 pad 4: Net-(D1-Pad2) -> /LED_TX
- U1 pad 24: unconnected-(U1-Pad24) -> /LED_TX
- U1 pad 3: +3V3 -> Net-(U1-Pad3)
- U1 pad 7: /LED_TX -> unconnected-(U1-Pad7)
- U5 pad 4: unconnected-(U5-Pad4) -> Earth
- U5 pad 5: unconnected-(U5-Pad4) -> Earth
Routing:
- net /LED_TX: track 27.5 -> 4.22 mm
- net +3V3: track 44.3 -> 57.1 mm, vias 1 -> 4
- net +5V: track 24.7 -> 33.8 mm
- net Net-(D2-Pad2): track 0.00 -> 9.14 mm
- net Net-(D1-Pad2): track 8.62 -> 0.00 mm
- net Net-(U1-Pad3): track 0.00 -> 8.47 mm
- net /BOOTLOADER: track 8.05 -> 12.1 mm
- net /BUZZER: track 5.54 -> 1.86 mm
- net /SCL: track 28.3 -> 31.6 mm
- net /USER_RTS: track 33.7 -> 36.9 mm, vias 3 -> 2
- net /SDA: track 11.0 -> 14.1 mm
- net Earth: track 72.5 -> 74.9 mm, vias 30 -> 29
- net unconnected-(U5-Pad4): track 2.15 -> 0.00 mm
- net /PYRO_1: track 37.3 -> 36.0 mm
- net /PYRO_3: track 37.9 -> 36.9 mm
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Other:
- board text added: "RESET"

Commit message: pre esp32 pico
Parts:
- added R10: 10k, Resistor_SMD:R_0603_1608Metric, B.Cu at (241.1, 128.8)
- added R11: 10k, Resistor_SMD:R_0603_1608Metric, B.Cu at (238.3, 128.0)
- added R12: 10k, Resistor_SMD:R_0603_1608Metric, B.Cu at (238.3, 125.0)
- added R13: 10k, Resistor_SMD:R_0603_1608Metric, B.Cu at (238.3, 121.9)
- added R9: 2k2, Resistor_SMD:R_0603_1608Metric, B.Cu at (229.9, 90.5)
- moved H1 0.27 mm to (215.0, 118.0)
- moved H3 0.27 mm to (241.0, 118.0)
- moved H2 0.23 mm to (241.0, 92.0)
- moved H4 0.21 mm to (215.0, 92.0)
Connections:
- J2 pad 1: +5V -> /USER_CTS
- J2 pad 2: /USER_RX -> /USER_RTS
- J2 pad 3: /USER_TX -> Earth
- J2 pad 4: Earth -> /USER_TX
- J2 pad 5: /USER_RTS -> /USER_RX
- J2 pad 6: /USER_CTS -> +5V
- U2 pad 12: unconnected-(U2-Pad12) -> Net-(U2-Pad12)
- U2 pad 16: unconnected-(U2-Pad16) -> Net-(U2-Pad12)
Routing:
- net /SERVO_1: track 23.0 -> 61.3 mm, vias 1 -> 2
- net /USER_CTS: track 36.9 -> 22.5 mm
- net /SERVO_2: track 26.0 -> 37.1 mm
- net Earth: track 74.9 -> 85.6 mm
- net /USER_RX: track 29.2 -> 36.1 mm
- net /SERVO_3: track 28.3 -> 34.2 mm
- net Net-(U2-Pad12): track 0.00 -> 4.27 mm, vias 0 -> 2
- net /USER_RTS: track 36.9 -> 33.0 mm
- net /SERVO_4: track 31.6 -> 34.4 mm
- net +3V3: track 57.1 -> 59.7 mm, vias 4 -> 3
- net +5V: track 33.8 -> 32.3 mm
- net Net-(BZ1-Pad2): track 5.68 -> 4.71 mm
- net /USER_TX: track 32.7 -> 33.4 mm
Other:
- board text added: "ESP_CONTROLLER DECEMBER-2022"
- board text removed: "ESP_CONTROLLER JULY-2022"
