File: schematic/esp_controller.kicad_sch (KiCad schematic)
At the start: 38 parts, among them J1 xt30, J2 jst_sh 6, J3 Conn_01x03, J4 Conn_01x03, J5 Conn_01x03, J6 Conn_01x03, J7 Screw_Terminal_01x06, Q1 FDN359BN, Q2 FDN359BN, Q3 FDN359BN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

Commit message: pcb second revision
Parts:
- added R6, R7: 2k2, Resistor_SMD:R_0603_1608Metric, symbol Device:R_Small
- added R8: 10k, Resistor_SMD:R_0603_1608Metric, symbol Device:R_Small
- added SW2: SW_SPST, Connector_PinHeader_1.27mm:PinHeader_1x02_P1.27mm_Vertical, symbol Switch:SW_SPST
- R2: value 2.2k -> 2k2
- SW1: footprint Connector_PinHeader_2.54mm:PinHeader_1x02_P2.54mm_Vertical -> Connector_PinHeader_1.27mm:PinHeader_1x02_P1.27mm_Vertical
- renumbered D2 to D1, D1 to D2
Connections:
- net +3V3: now also R6.2, R7.2, R8.1; no longer U1.3 (EN)
- net Earth: now also U5.4 (CSB), U5.5 (CSB), SW2.1 (A)
- net LED_TX: now also U1.24 (IO2); no longer U1.7 (IO35)
- net SCL: now also R7.1
- net SDA: now also R6.1
- new net: R8.2, SW2.2 (B), U1.3 (EN)
- no-connect marks 21 -> 20
Other:
- note removed: "OOPS no pull ups"
- moved on the sheet: C4, U5

Commit message: pre esp32 pico
Parts:
- added R10, R11, R12, R13: 10k, Resistor_SMD:R_0603_1608Metric, symbol Device:R_Small
- added R9: 2k2, Resistor_SMD:R_0603_1608Metric, symbol Device:R_Small
Connections:
- net +3V3: now also R9.2
- net +5V: now also J2.6 (Pin_6); no longer J2.1 (Pin_1)
- net Earth: now also J2.3 (Pin_3), R10.2, R11.2, R12.2, R13.2; no longer J2.4 (Pin_4)
- net SERVO_1: now also R10.1, R9.1
- net SERVO_2: now also R11.1
- net SERVO_3: now also R12.1
- net SERVO_4: now also R13.1
- net USER_CTS: now also J2.1 (Pin_1); no longer J2.6 (Pin_6)
- net USER_RTS: now also J2.2 (Pin_2); no longer J2.5 (Pin_5)
- net USER_RX: now also J2.5 (Pin_5); no longer J2.2 (Pin_2)
- net USER_TX: now also J2.4 (Pin_4); no longer J2.3 (Pin_3)
- net at U2.12 (INT3): now also U2.16 (INT1)
- no-connect marks 20 -> 19
Other:
- note added: "NCS standard"
- note added: "accel & gyro sync"
- moved on the sheet: C5, J2, J3, J4, J5, J6
